Commit message: checkpoint before playing with urdf

File: src/multi_robot_arm/urdf/lidar.xacro (robot description, xacro)
@@ -4,5 +4,5 @@
         <parent link="chassis_link"/>
         <child link="laser_frame"/>
-        <origin xyz="0.3 0 0.25" rpy="0 0 0"/>
+        <origin xyz="0.3 0 0.3" rpy="0 0 0"/>
     </joint>
     <link name="laser_frame">
@@ -43,5 +43,5 @@
                 <range>
                     <min>0.1</min>
-                    <max>12</max>
+                    <max>20</max>
                 </range>
             </ray>
