Commit message: morning commit

File: src/multi_robot_arm/urdf/logotest.xacro (robot description, xacro)
@@ -179,11 +179,4 @@
 		<origin xyz="0 0 0.16" rpy="0 0 0" />
 	</joint>
-<!-- ............................. RWTH LOGO ........................................ -->
-	<visual>
-			<origin xyz="0 0 0" rpy="0 0 0" />
-			<geometry>
-				<mesh filename="file://$(find multi_robot_arm)/meshes/logo.dae"/>
-			</geometry>
-	</visual>
 <!-- ............................. CONVEYOR ........................................ -->
 <xacro:if value="$(arg conveyor_enabled)">
