Commit message: fuer peter

File: src/multi_robot_arm/urdf/gazebo.xacro (robot description, xacro)
@@ -1,4 +1,4 @@
 <?xml version="1.0"?>
-<robot xmlns:xacro="http://www.ros.org/wiki/xacro" name="bcr_bot">
+<robot xmlns:xacro="http://www.ros.org/wiki/xacro" name="bot1">
 <gazebo>
 	<static>false</static>
@@ -9,5 +9,5 @@
 		<ros>
 			<namespace>$(arg robot_namespace)</namespace>
-			<remapping>cmd_vel:=cmd_vel</remapping>
+		  	<remapping>cmd_vel:=cmd_vel</remapping>
 			<remapping>odom:=odom</remapping>
 		</ros>
@@ -18,11 +18,9 @@
 		<wheel_separation>${traction_track_width+traction_wheel_width-0.01}</wheel_separation>
 		<wheel_diameter>${2*traction_wheel_radius+0.01}</wheel_diameter>
-		<robot_base_frame>base_link</robot_base_frame>
+		<robot_base_frame>$(arg robot_namespace)/base_footprint</robot_base_frame>
 		<max_wheel_torque>${traction_max_wheel_torque}</max_wheel_torque>
-		<command_topic>cmd_vel</command_topic>
-		<odometry_topic>$(arg wheel_odom_topic)</odometry_topic>
-		<odometry_frame>odom</odometry_frame>
-		<publish_odom_tf>$(arg publish_wheel_odom_tf)</publish_odom_tf>
-		<publish_wheel_tf>true</publish_wheel_tf>
+		<odometry_frame>$(arg robot_namespace)/odom</odometry_frame>
+		<publish_odom_tf>true</publish_odom_tf>
+		<publish_wheel_tf>false</publish_wheel_tf>
 		<publish_odom>true</publish_odom>
 		<max_wheel_acceleration>5.0</max_wheel_acceleration>
@@ -50,18 +48,4 @@
 </gazebo>
 <!--............................... Ground truth PLUGIN .............................-->
-<gazebo>
-	<plugin name="p3d_base_controller" filename="libgazebo_ros_p3d.so">
-		<ros>
-			<!-- Add namespace and remap the default topic -->
-			<namespace>$(arg robot_namespace)</namespace>
-			<remapping>odom:=p3d_ground_truth</remapping>
-		</ros>
-		<always_on>true</always_on>
-		<update_rate>30.0</update_rate>
-		<body_name>base_link</body_name>
-		<gaussian_noise>0.00</gaussian_noise>
-		<frame_name>$(arg ground_truth_frame)</frame_name>
-	</plugin>
-</gazebo>
 <!-- ........................... 2D LIDAR PLUGIN ................................... -->
 <xacro:if value="$(arg two_d_lidar_enabled)">

File: src/multi_robot_arm/urdf/logotest.xacro (robot description, xacro)
@@ -28,5 +28,5 @@
 <xacro:property name="camera_height"               value="0.10"/>
 <xacro:property name="camera_horizontal_fov"       value="60"/>
-<xacro:arg      name="robot_namespace"             default=""/>
+<xacro:arg      name="robot_namespace"             default="bot1"/>
 <xacro:arg      name="wheel_odom_topic"            default="odom" />
 <xacro:arg      name="camera_enabled"              default="false" />
@@ -43,20 +43,16 @@
 <xacro:include filename="$(find multi_robot_arm)/urdf/macros.xacro"/>
 <xacro:include filename="$(find multi_robot_arm)/urdf/inertial_macros.xacro"/>
-<xacro:include filename="$(find multi_robot_arm)/urdf/lidar.xacro"/>
+<!-- <xacro:include filename="$(find multi_robot_arm)/urdf/lidar.xacro"/> -->
 <xacro:if value="$(arg sim_gazebo)">
 	<xacro:include filename="$(find multi_robot_arm)/urdf/gazebo.xacro"/>
 </xacro:if>
-<xacro:if value="$(arg sim_gz)">
-	<xacro:include filename="$(find multi_robot_arm)/urdf/gz.xacro"/>
-</xacro:if>
 <!-- ................................ BASE LINK .................................. -->
 <link name="base_link"/>
- <joint name="base_footprint_joint" type="fixed">
-    <parent link="base_link"/>
-    <child link="base_footprint"/>
-	    <origin xyz="0 0 0" rpy="0 0 0"/>
- </joint>
-<link name="base_footprint">
-</link>
+<link name="base_footprint"/>
+<joint name="base_joint" type="fixed">
+    <parent link="base_footprint"/>
+    <child link = "base_link"/>
+    <pose>0.0 0.0 0.0 0 0 0</pose>
+</joint>
 <link name="chassis_link">
 	<collision>
